Commit message: added lidar and camera

File: description/common_properties.xacro (robot description, xacro)
@@ -15,4 +15,7 @@
     <material name="orange">
         <color rgba="1 0.3 0.1 1" />
+    </material>
+    <material name="red">
+        <color rgba="1 0 0 1" />
     </material>
     <xacro:macro name="box_inertia" params="m l w h xyz rpy">

File: description/pickup_bot.urdf.xacro (robot description, xacro)
@@ -4,3 +4,5 @@
     <xacro:include filename="mobile_base.xacro" />
     <xacro:include filename="mobile_base_gazebo.xacro" />
+    <xacro:include filename="lidar.xacro" />
+    <xacro:include filename="camera.xacro" />
 </robot>
